File: electrical/tank.sch (EAGLE design)
At the start: 0 parts

Commit message: Added IC's and passives to schematic, library
Parts:
- added CIN: 1m, rcl:CPOL-USE3.5-10
- added CO: 560u, rcl:CPOL-USE5-13
- added CT: 470p, eagle-ltspice:CC0402
- added ILIM: 15, tank:RR0603
- added L1: 10u, tank:AIUR-06-100K
- added R1: 2.2k, resistor:R-US_R0402
- added R2: 41.2k, resistor:R-US_R0805
- added RSENSE: 0.04, tank:RR2010
- added U$1: SSC53L, tank:SSC53L
- added U1: MC33063ADR, tank:MC33063ADR
Connections:
- new net 0: CIN.-, CO.-, CT.2, R1.1, U1.SWITCHEMITTER
- new net IC: ILIM.2, U1.DRIVERCOLLECTOR
- new net LIN: ILIM.1, L1.1, RSENSE.2, U1.IPK
- new net LOUT: L1.2, U$1.A, U1.SWITCHCOLLECTOR
- new net N$1: R1.2, R2.1, U1.COMPARATORINVERTINGINPUT
- new net N$2: CT.1, U1.TIMINGCAPACITOR
- new net VCC: CIN.+, RSENSE.1, U1.VCC
- new net VOUT: CO.+, R2.2, U$1.C
